Commit message: Setup collisions, inertia and bone links correctly for phobos

File: model/phobos/urdf/robodog.urdf (robot description, URDF)
Before this commit: robot robodog, 14 links, 13 joints
Links:
- link back_left_bot_leg_link: mass None -> 0.00100; geometry collision cylinder length=0.14640 radius=0.16016; collision cylinder length=0.37440 radius=0.10289
- link back_left_mid_leg_link: mass None -> 0.00100; geometry collision cylinder length=0.15862 radius=0.14306; visual mesh filename=../meshes/stl/back_left_top_leg_mesh.015.stl scale=1.00000 1.00000 1.00000
- link back_left_top_leg_link: mass None -> 0.00100
- link back_right_bot_leg_link: mass None -> 0.00100; geometry collision cylinder length=0.14640 radius=0.16016; collision cylinder length=0.37440 radius=0.10289
- link back_right_mid_leg_link: mass None -> 0.00100; geometry collision cylinder length=0.15862 radius=0.14306; visual mesh filename=../meshes/stl/back_left_top_leg_mesh.035.stl scale=1.00000 1.00000 1.00000
- link back_right_top_leg_link: mass None -> 0.00100; geometry collision cylinder length=0.77385 radius=0.22085; visual mesh filename=../meshes/stl/back_left_top_leg_mesh.020.stl scale=1.00000 1.00000 1.00000
- link front_left_bot_leg_link: mass None -> 0.00100; geometry collision cylinder length=0.14640 radius=0.16016; collision cylinder length=0.38831 radius=0.10671
- link front_left_mid_leg_link: mass None -> 0.00100; geometry collision cylinder length=0.17878 radius=0.14307; visual mesh filename=../meshes/stl/back_left_top_leg_mesh.004.stl scale=1.00000 1.00000 1.00000
- link front_left_top_leg_link: mass None -> 0.00100; geometry collision cylinder length=1.01216 radius=0.21890; visual mesh filename=../meshes/stl/back_left_top_leg_mesh.012.stl scale=1.00000 1.00000 1.00000
- link front_right_bot_leg_link: mass None -> 0.00100; geometry collision cylinder length=0.14640 radius=0.16016; collision cylinder length=0.38831 radius=0.10671
- link front_right_mid_leg_link: mass None -> 0.00100; geometry collision cylinder length=0.17878 radius=0.14307; visual mesh filename=../meshes/stl/back_left_top_leg_mesh.024.stl scale=1.00000 1.00000 1.00000
- link front_right_top_leg_link: mass None -> 0.00100; geometry collision cylinder length=1.01216 radius=0.21890; visual mesh filename=../meshes/stl/back_left_top_leg_mesh.033.stl scale=1.00000 1.00000 1.00000
- link main_link: mass 1.00000 -> 0.00100
Joints:
- joint back_left_bot_leg_link_joint: limit lower=-3.14000 upper=3.14000 effort=0.00000 velocity=0.00000 -> lower=-1.04720 upper=2.79253 effort=0.00000 velocity=0.00000; origin xyz=0.35179 0.41990 -0.00481 rpy=0.00000 0.00000 0.00000 -> xyz=0.35155 0.41990 -0.01402 rpy=0.00000 0.00000 0.00000
- joint back_left_mid_leg_link_joint: limit lower=-3.14000 upper=3.14000 effort=0.00000 velocity=0.00000 -> lower=-1.57080 upper=0.87266 effort=0.00000 velocity=1.04720; origin xyz=0.07103 0.13951 -0.49515 rpy=-1.57080 -0.00000 0.00000 -> xyz=0.07465 0.13760 -0.49515 rpy=-1.57079 0.00000 0.00000
- joint back_left_top_leg_link_joint: origin xyz=0.33081 0.34784 -0.07472 rpy=-1.57080 1.54462 3.14159 -> xyz=0.33081 0.34784 -0.07472 rpy=1.57079 1.57080 0.00000
- joint back_right_bot_leg_link_joint: limit lower=-3.14000 upper=3.14000 effort=0.00000 velocity=0.00000 -> lower=-2.79253 upper=1.04720 effort=0.00000 velocity=1.04720; origin xyz=-0.35179 0.41990 -0.00481 rpy=0.00000 0.00000 -0.00000 -> xyz=-0.35155 0.41990 -0.01402 rpy=-0.00000 0.00000 -0.00000
- joint back_right_mid_leg_link_joint: limit lower=-3.14000 upper=3.14000 effort=0.00000 velocity=0.00000 -> lower=-0.87266 upper=1.57080 effort=0.00000 velocity=1.04720; origin xyz=-0.06860 0.14163 -0.49515 rpy=-1.57079 -0.00000 -0.01697 -> xyz=-0.07698 0.13632 -0.49515 rpy=-1.57079 0.00000 0.01697
- joint back_right_top_leg_link_joint: origin xyz=-0.32753 0.34784 -0.07476 rpy=-1.57080 -1.54462 3.14159 -> xyz=-0.33081 0.34784 -0.07472 rpy=1.57079 -1.57080 0.00000
- joint front_left_bot_leg_link_joint: limit lower=-3.14000 upper=3.14000 effort=0.00000 velocity=0.00000 -> lower=-1.04720 upper=2.79253 effort=0.00000 velocity=0.00000; origin xyz=0.32430 0.44600 0.07792 rpy=-0.00000 0.00000 -0.08125 -> xyz=0.28599 0.47085 0.08165 rpy=0.00000 0.00000 0.00000
- joint front_left_mid_leg_link_joint: limit lower=-3.14000 upper=3.14000 effort=0.00000 velocity=0.00000 -> lower=-1.57080 upper=0.87266 effort=0.00000 velocity=1.04720; origin xyz=0.07403 0.07293 -0.28308 rpy=-1.57080 0.00000 -0.00000 -> xyz=0.07307 0.07389 -0.28308 rpy=-1.57080 0.00000 0.00000
- joint front_left_top_leg_link_joint: origin xyz=0.33081 -1.00714 -0.07472 rpy=-1.57082 1.56207 3.14159 -> xyz=0.33081 -1.00714 -0.07472 rpy=1.57080 1.57080 0.00000
- joint front_right_bot_leg_link_joint: limit lower=-3.14000 upper=3.14000 effort=0.00000 velocity=0.00000 -> lower=-2.79253 upper=1.04720 effort=0.00000 velocity=0.00000; origin xyz=-0.28704 0.47085 0.04169 rpy=-0.00000 0.00000 -0.00000 -> xyz=-0.28599 0.47085 0.08165 rpy=-0.00000 0.00000 -0.00000
- joint front_right_mid_leg_link_joint: limit lower=-3.14000 upper=3.14000 effort=0.00000 velocity=0.00000 -> lower=-0.87266 upper=1.57080 effort=0.00000 velocity=1.04720; origin xyz=-0.07415 0.10999 -0.28308 rpy=-1.57080 -0.00000 0.00136 -> xyz=-0.07297 0.07399 -0.28308 rpy=-1.57080 0.00000 -0.00136
- joint front_right_top_leg_link_joint: origin xyz=-0.32753 -1.00714 -0.07476 rpy=-1.57082 -1.56207 -3.14159 -> xyz=-0.33081 -1.00714 -0.07472 rpy=1.57080 -1.57080 0.00000

Commit message: Modifications to back leg, phobos meshes

File: model/phobos/urdf/robodog.urdf (robot description, URDF)
Before this commit: robot robodog, 14 links, 13 joints
Links:
- added link back_left_leg_foot_link; collision sphere radius=0.10444; visual mesh filename=../meshes/stl/back_left_top_leg_mesh.012.stl scale=1.00000 1.00000 1.00000
- added link back_right_leg_foot_link; collision sphere radius=0.10444; visual mesh filename=../meshes/stl/back_left_top_leg_mesh.013.stl scale=1.00000 1.00000 1.00000
- added link front_left_leg_foot_link; collision sphere radius=0.10458; visual mesh filename=../meshes/stl/back_left_top_leg_mesh.014.stl scale=1.00000 1.00000 1.00000
- added link front_right_leg_foot_link; collision sphere radius=0.10458; visual mesh filename=../meshes/stl/back_left_top_leg_mesh.015.stl scale=1.00000 1.00000 1.00000
- link back_left_bot_leg_link: mass 0.00100 -> 1.00000; geometry collision cylinder length=0.14640 radius=0.16016; collision cylinder length=0.37440 radius=0.10289
- link back_left_mid_leg_link: mass 0.00100 -> 1.00000; geometry collision cylinder length=0.15862 radius=0.14306; visual mesh filename=../meshes/stl/back_left_top_leg_mesh.004.stl scale=1.00000 1.00000 1.00000
- link back_left_top_leg_link: mass 0.00100 -> 1.00000
- link back_right_bot_leg_link: mass 0.00100 -> 1.00000; geometry collision cylinder length=0.14640 radius=0.16016; collision cylinder length=0.37440 radius=0.10289
- link back_right_mid_leg_link: mass 0.00100 -> 1.00000; geometry collision cylinder length=0.15862 radius=0.14306; visual mesh filename=../meshes/stl/back_left_top_leg_mesh.010.stl scale=1.00000 1.00000 1.00000
- link back_right_top_leg_link: mass 0.00100 -> 1.00000; geometry collision cylinder length=0.77385 radius=0.22085; visual mesh filename=../meshes/stl/back_left_top_leg_mesh.006.stl scale=1.00000 1.00000 1.00000
- link front_left_bot_leg_link: mass 0.00100 -> 1.00000; geometry collision cylinder length=0.15749 radius=0.16262; collision cylinder length=0.38831 radius=0.10671
- link front_left_mid_leg_link: mass 0.00100 -> 1.00000; geometry collision cylinder length=0.17878 radius=0.14307; visual mesh filename=../meshes/stl/back_left_top_leg_mesh.001.stl scale=1.00000 1.00000 1.00000
- link front_left_top_leg_link: mass 0.00100 -> 1.00000; geometry collision cylinder length=1.01216 radius=0.21890; visual mesh filename=../meshes/stl/back_left_top_leg_mesh.003.stl scale=1.00000 1.00000 1.00000
- link front_right_bot_leg_link: mass 0.00100 -> 1.00000; geometry collision cylinder length=0.15749 radius=0.16262; collision cylinder length=0.38831 radius=0.10671
- link front_right_mid_leg_link: mass 0.00100 -> 1.00000; geometry collision cylinder length=0.17878 radius=0.14307; visual mesh filename=../meshes/stl/back_left_top_leg_mesh.007.stl scale=1.00000 1.00000 1.00000
- link front_right_top_leg_link: mass 0.00100 -> 1.00000; geometry collision cylinder length=1.01216 radius=0.21890; visual mesh filename=../meshes/stl/back_left_top_leg_mesh.009.stl scale=1.00000 1.00000 1.00000
- link main_link: mass 0.00100 -> 1.00000
Joints:
- added joint back_left_ball_collision_link_joint: type fixed, parent front_left_bot_leg_link, child front_left_leg_foot_link, origin xyz=0.57902 -0.34558 -0.02243 rpy=-3.14159 -1.57080 0.00000
- added joint back_right_ball_collision_link_joint: type fixed, parent front_right_bot_leg_link, child front_right_leg_foot_link, origin xyz=-0.57920 -0.34558 -0.02371 rpy=-3.14159 1.56944 -0.00000
- added joint front_left_ball_collision_link_joint: type fixed, parent back_left_bot_leg_link, child back_left_leg_foot_link, origin xyz=0.48243 -0.47826 0.00556 rpy=-3.14159 -1.57080 0.00000
- added joint front_right_ball_collision_link_joint: type fixed, parent back_right_bot_leg_link, child back_right_leg_foot_link, origin xyz=-0.48011 -0.47826 0.02096 rpy=0.00000 1.55383 3.14159
